Commit message: feat: 5축 키보드 텔레옵 완성
5축 URDF/메시를 반영하고 텔레옵 조인트를 joint_1..joint_5로 확장한다.

RViz 시뮬레이션과 실제 Dynamixel 목표 위치에 동일한 관절 제한을 적용한다.

README, CLAUDE, AGENTS 문서를 현재 브랜치 범위와 테스트 절차에 맞게 갱신한다.

File: ros2_ws/src/robot_arm_description/urdf/robot_arm.urdf (robot description, URDF)
Before this commit: robot robot_arm, 30 links, 29 joints
Links:
- removed link Adapter_A_1
- removed link Adapter_A_1_1
- removed link Adapter_B_1
- removed link Adapter_B_1_1_1
- removed link Adapter_b_1_1
- removed link Bottom_Cylinder_1
- removed link Bottom_top_1
- removed link GearBox1_1
- removed link GearBox2_1
- removed link Link1_1
- removed link Link1_1_1
- removed link Link2Bridge2_1
- removed link Link2Bridge_1
- removed link Link2_1
- removed link Link2_1_1
- removed link Link3Bridge2_1
- removed link Link3Bridge_1
- removed link Link3_1
- removed link Link3_1_1
- removed link Link4_1
- removed link Link4_1_1
- removed link Link5_1_1
- removed link Link_5_1
- removed link Motor0_1
- removed link Motor1_1
- removed link Motor2_1
- removed link Motor_1
- removed link Plug_1
- removed link _Plug2_1
- added link Component38_1, mass 0.5585472030657777; collision mesh filename=package://robot_arm_description/meshes/Component38_1.stl scale=0.001 0.001 0.001; visual mesh filename=package://robot_arm_description/meshes/Component38_1.stl scale=0.001 0.001 0.001
- added link Component40_1, mass 0.6121227780764895; collision mesh filename=package://robot_arm_description/meshes/Component40_1.stl scale=0.001 0.001 0.001; visual mesh filename=package://robot_arm_description/meshes/Component40_1.stl scale=0.001 0.001 0.001
- added link XL430_T_1, mass 0.34622507558019666; collision mesh filename=package://robot_arm_description/meshes/XL430_T_1.stl scale=0.001 0.001 0.001; visual mesh filename=package://robot_arm_description/meshes/XL430_T_1.stl scale=0.001 0.001 0.001
- added link adapter_1, mass 0.037276333994375375; collision mesh filename=package://robot_arm_description/meshes/adapter_1.stl scale=0.001 0.001 0.001; visual mesh filename=package://robot_arm_description/meshes/adapter_1.stl scale=0.001 0.001 0.001
- added link adapter_a_1, mass 0.09838512042156757; collision mesh filename=package://robot_arm_description/meshes/adapter_a_1.stl scale=0.001 0.001 0.001; visual mesh filename=package://robot_arm_description/meshes/adapter_a_1.stl scale=0.001 0.001 0.001
- added link adapter_a__1__1, mass 0.09838512042156751; collision mesh filename=package://robot_arm_description/meshes/adapter_a__1__1.stl scale=0.001 0.001 0.001; visual mesh filename=package://robot_arm_description/meshes/adapter_a__1__1.stl scale=0.001 0.001 0.001
- added link adapter_b_1, mass 0.0383693503096125; collision mesh filename=package://robot_arm_description/meshes/adapter_b_1.stl scale=0.001 0.001 0.001; visual mesh filename=package://robot_arm_description/meshes/adapter_b_1.stl scale=0.001 0.001 0.001
- added link adapter_b__1__1, mass 0.1507674746734739; collision mesh filename=package://robot_arm_description/meshes/adapter_b__1__1.stl scale=0.001 0.001 0.001; visual mesh filename=package://robot_arm_description/meshes/adapter_b__1__1.stl scale=0.001 0.001 0.001
- added link adapter_b__1___1__1, mass 0.0836288961017048; collision mesh filename=package://robot_arm_description/meshes/adapter_b__1___1__1.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 scale=0.001 0.001 0.001; visual mesh filename=package://robot_arm_description/meshes/adapter_b__1___1__1.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 scale=0.001 0.001 0.001
- added link base_plate_1, mass 0.7527923586440036; collision mesh filename=package://robot_arm_description/meshes/base_plate_1.stl scale=0.001 0.001 0.001; visual mesh filename=package://robot_arm_description/meshes/base_plate_1.stl scale=0.001 0.001 0.001
- added link bottom_1, mass 0.12615164501277876; collision mesh filename=package://robot_arm_description/meshes/bottom_1.stl scale=0.001 0.001 0.001; visual mesh filename=package://robot_arm_description/meshes/bottom_1.stl scale=0.001 0.001 0.001
- added link cap2_1, mass 0.12724315500067693; collision mesh filename=package://robot_arm_description/meshes/cap2_1.stl scale=0.001 0.001 0.001; visual mesh filename=package://robot_arm_description/meshes/cap2_1.stl scale=0.001 0.001 0.001
- added link cap_1, mass 0.1272431550006768; collision mesh filename=package://robot_arm_description/meshes/cap_1.stl scale=0.001 0.001 0.001; visual mesh filename=package://robot_arm_description/meshes/cap_1.stl scale=0.001 0.001 0.001
- added link connector_1__1, mass 0.14836014599953082; collision mesh filename=package://robot_arm_description/meshes/connector_1__1.stl scale=0.001 0.001 0.001; visual mesh filename=package://robot_arm_description/meshes/connector_1__1.stl scale=0.001 0.001 0.001
- added link gearbox1_1, mass 2.039024001006148; collision mesh filename=package://robot_arm_description/meshes/gearbox1_1.stl scale=0.001 0.001 0.001; visual mesh filename=package://robot_arm_description/meshes/gearbox1_1.stl scale=0.001 0.001 0.001
- added link gearbox1__1__1, mass 2.0338757908094958; collision mesh filename=package://robot_arm_description/meshes/gearbox1__1__1.stl scale=0.001 0.001 0.001; visual mesh filename=package://robot_arm_description/meshes/gearbox1__1__1.stl scale=0.001 0.001 0.001
- added link link1-1_1, mass 0.40614905152898423; collision mesh filename=package://robot_arm_description/meshes/link1-1_1.stl scale=0.001 0.001 0.001; visual mesh filename=package://robot_arm_description/meshes/link1-1_1.stl scale=0.001 0.001 0.001
- added link link1_1, mass 0.44759500853450696; collision mesh filename=package://robot_arm_description/meshes/link1_1.stl scale=0.001 0.001 0.001; visual mesh filename=package://robot_arm_description/meshes/link1_1.stl scale=0.001 0.001 0.001
- added link link1__1__1, mass 0.1900850226097608; collision mesh filename=package://robot_arm_description/meshes/link1__1__1.stl scale=0.001 0.001 0.001; visual mesh filename=package://robot_arm_description/meshes/link1__1__1.stl scale=0.001 0.001 0.001
- added link link2-1__3__1, mass 0.5733792760793044; collision mesh filename=package://robot_arm_description/meshes/link2-1__3__1.stl scale=0.001 0.001 0.001; visual mesh filename=package://robot_arm_description/meshes/link2-1__3__1.stl scale=0.001 0.001 0.001
- added link link2_1, mass 0.5760752094127702; collision mesh filename=package://robot_arm_description/meshes/link2_1.stl scale=0.001 0.001 0.001; visual mesh filename=package://robot_arm_description/meshes/link2_1.stl scale=0.001 0.001 0.001
- added link link2__1__1, mass 0.20741862160121777; collision mesh filename=package://robot_arm_description/meshes/link2__1__1.stl scale=0.001 0.001 0.001; visual mesh filename=package://robot_arm_description/meshes/link2__1__1.stl scale=0.001 0.001 0.001
- added link link2_leg2_1, mass 0.17597826669199707; collision mesh filename=package://robot_arm_description/meshes/link2_leg2_1.stl scale=0.001 0.001 0.001; visual mesh filename=package://robot_arm_description/meshes/link2_leg2_1.stl scale=0.001 0.001 0.001
- added link link2_leg_1, mass 0.22700261556158713; collision mesh filename=package://robot_arm_description/meshes/link2_leg_1.stl scale=0.001 0.001 0.001; visual mesh filename=package://robot_arm_description/meshes/link2_leg_1.stl scale=0.001 0.001 0.001
- added link link3-1_1, mass 0.8186445791058825; collision mesh filename=package://robot_arm_description/meshes/link3-1_1.stl scale=0.001 0.001 0.001; visual mesh filename=package://robot_arm_description/meshes/link3-1_1.stl scale=0.001 0.001 0.001
- added link link3_1, mass 0.8034510771086975; collision mesh filename=package://robot_arm_description/meshes/link3_1.stl scale=0.001 0.001 0.001; visual mesh filename=package://robot_arm_description/meshes/link3_1.stl scale=0.001 0.001 0.001
- added link link3_leg2_1, mass 0.2226363143753701; collision mesh filename=package://robot_arm_description/meshes/link3_leg2_1.stl scale=0.001 0.001 0.001; visual mesh filename=package://robot_arm_description/meshes/link3_leg2_1.stl scale=0.001 0.001 0.001
- added link link3_leg_1, mass 0.3308579843753697; collision mesh filename=package://robot_arm_description/meshes/link3_leg_1.stl scale=0.001 0.001 0.001; visual mesh filename=package://robot_arm_description/meshes/link3_leg_1.stl scale=0.001 0.001 0.001
- added link link4-1_1, mass 0.21082599155250997; collision mesh filename=package://robot_arm_description/meshes/link4-1_1.stl scale=0.001 0.001 0.001; visual mesh filename=package://robot_arm_description/meshes/link4-1_1.stl scale=0.001 0.001 0.001
- added link link4_1, mass 0.21082599155250994; collision mesh filename=package://robot_arm_description/meshes/link4_1.stl scale=0.001 0.001 0.001; visual mesh filename=package://robot_arm_description/meshes/link4_1.stl scale=0.001 0.001 0.001
- added link link5-1_1, mass 0.24038547715832267; collision mesh filename=package://robot_arm_description/meshes/link5-1_1.stl scale=0.001 0.001 0.001; visual mesh filename=package://robot_arm_description/meshes/link5-1_1.stl scale=0.001 0.001 0.001
- added link link5_1, mass 0.2576677637629673; collision mesh filename=package://robot_arm_description/meshes/link5_1.stl scale=0.001 0.001 0.001; visual mesh filename=package://robot_arm_description/meshes/link5_1.stl scale=0.001 0.001 0.001
- added link lower_cylinder_1, mass 2.7522236601038736; collision mesh filename=package://robot_arm_description/meshes/lower_cylinder_1.stl scale=0.001 0.001 0.001; visual mesh filename=package://robot_arm_description/meshes/lower_cylinder_1.stl scale=0.001 0.001 0.001
- added link module_connector_5axis_Component41_1, mass 1.9126732622839608; collision mesh filename=package://robot_arm_description/meshes/module_connector_5ax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 scale=0.001 0.001 0.001; visual mesh filename=package://robot_arm_description/meshes/module_connector_5ax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 scale=0.001 0.001 0.001
- added link motor0_1, mass 0.664027798614862; collision mesh filename=package://robot_arm_description/meshes/motor0_1.stl scale=0.001 0.001 0.001; visual mesh filename=package://robot_arm_description/meshes/motor0_1.stl scale=0.001 0.001 0.001
- added link motor1_1, mass 0.6640277986148614; collision mesh filename=package://robot_arm_description/meshes/motor1_1.stl scale=0.001 0.001 0.001; visual mesh filename=package://robot_arm_description/meshes/motor1_1.stl scale=0.001 0.001 0.001
- added link motor2_1, mass 0.6620566191194474; collision mesh filename=package://robot_arm_description/meshes/motor2_1.stl scale=0.001 0.001 0.001; visual mesh filename=package://robot_arm_description/meshes/motor2_1.stl scale=0.001 0.001 0.001
- added link motor_1, mass 0.6640277986148609; collision mesh filename=package://robot_arm_description/meshes/motor_1.stl scale=0.001 0.001 0.001; visual mesh filename=package://robot_arm_description/meshes/motor_1.stl scale=0.001 0.001 0.001
- added link powertrain_1, mass 0.0024661502330680955; collision mesh filename=package://robot_arm_description/meshes/powertrain_1.stl scale=0.001 0.001 0.001; visual mesh filename=package://robot_arm_description/meshes/powertrain_1.stl scale=0.001 0.001 0.001
- added link top_1, mass 0.11483450819161148; collision mesh filename=package://robot_arm_description/meshes/top_1.stl scale=0.001 0.001 0.001; visual mesh filename=package://robot_arm_description/meshes/top_1.stl scale=0.001 0.001 0.001
Joints:
- removed joint Rigid 23
- removed joint Rigid 42
- removed joint Rigid 48
- removed joint Rigid 5
- removed joint Rigid 54
- removed joint Rigid 55
- removed joint Rigid 56
- removed joint Rigid 57
- removed joint Rigid 58
- removed joint Rigid 59
- removed joint Rigid 60
- removed joint Rigid 61
- added joint Rigid 20: type fixed, parent base_link, child motor0_1, origin xyz=0.0 0.0 0.004 rpy=0 0 0
- added joint Rigid 24: type fixed, parent base_plate_1, child link1-1_1, origin xyz=0.0 -0.01 0.0085 rpy=0 0 0
- added joint Rigid 25: type fixed, parent base_plate_1, child link1_1, origin xyz=0.0 -0.01 0.0085 rpy=0 0 0
- added joint Rigid 26: type fixed, parent link1-1_1, child gearbox1_1, origin xyz=-0.06215 0.004643 0.06 rpy=0 0 0
- added joint Rigid 27: type fixed, parent gearbox1_1, child adapter_a_1, origin xyz=0.0675 -0.005731 0.0 rpy=0 0 0
- added joint Rigid 28: type fixed, parent adapter_a_1, child motor_1, origin xyz=0.0103 0.005544 -0.0045 rpy=0 0 0
- added joint Rigid 30: type fixed, parent adapter_b_1, child Component40_1, origin xyz=0.0148 0.0 0.0 rpy=0 0 0
- added joint Rigid 31: type fixed, parent Component40_1, child link2_1, origin xyz=0.002 0.15 -0.001 rpy=0 0 0
- added joint Rigid 32: type fixed, parent link2_1, child adapter_b__1__1, origin xyz=-0.002 0.143 0.061 rpy=0 0 0
- added joint Rigid 33: type fixed, parent link2_1, child link2_leg2_1, origin xyz=0.002 0.013819 -0.047 rpy=0 0 0
- added joint Rigid 34: type fixed, parent Component40_1, child link2_leg_1, origin xyz=0.002 0.135652 0.049 rpy=0 0 0
- added joint Rigid 35: type fixed, parent link2_leg_1, child Component38_1, origin xyz=-0.1586 0.025 0.0 rpy=0 0 0
- added joint Rigid 36: type fixed, parent link2_leg_1, child link2-1__3__1, origin xyz=-0.1586 0.0 0.0 rpy=0 0 0
- added joint Rigid 37: type fixed, parent link2-1__3__1, child cap_1, origin xyz=-0.002 -0.135652 -0.049 rpy=0 0 0
- added joint Rigid 38: type fixed, parent adapter_b__1__1, child motor1_1, origin xyz=-0.0303 0.0 0.0 rpy=0 0 0
- added joint Rigid 39: type fixed, parent motor1_1, child adapter_a__1__1, origin xyz=-0.044 0.0 0.0 rpy=0 0 0
- added joint Rigid 40: type fixed, parent adapter_a__1__1, child gearbox1__1__1, origin xyz=-0.0407 0.0 0.0 rpy=0 0 0
- added joint Rigid 44: type fixed, parent link3_1, child link3_leg_1, origin xyz=0.0 -0.10674 0.108 rpy=0 0 0
- added joint Rigid 66: type fixed, parent top_1, child link1__1__1, origin xyz=0.0819 0.0 0.0 rpy=0 0 0
- added joint Rigid 71: type fixed, parent link2__1__1, child XL430_T_1, origin xyz=0.01505 -0.100544 -0.00025 rpy=0 0 0
- added joint Rigid 73: type fixed, parent connector_1__1, child module_connector_5axis_Component41_1, origin xyz=0.0 -0.0051 0.0 rpy=0 0 0
- added joint joint_4: type revolute, parent link5_1, child adapter_1, origin xyz=0.0001 -0.068917 0.0045 rpy=0 0 0, axis -1.0 0.0 0.0, limit lower=-1.570796 upper=1.570796 effort=100 velocity=100
- added joint joint_5: type revolute, parent XL430_T_1, child connector_1__1, origin xyz=0.0309 0.001644 -0.00525 rpy=0 0 0, axis -0.0 -1.0 0.0, limit lower=-3.141593 upper=3.141593 effort=100 velocity=100
- joint Rigid 21: child Bottom_Cylinder_1 -> lower_cylinder_1; origin xyz=0.0 0.01 -0.0005 rpy=0 0 0 -> xyz=0.0 0.0 0.004 rpy=0 0 0
- joint Rigid 22: child Link1_1 -> powertrain_1; origin xyz=0.0 0.0 0.004 rpy=0 0 0 -> xyz=0.0 0.0 0.0465 rpy=0 0 0; parent Bottom_top_1 -> lower_cylinder_1
- joint Rigid 43: child Motor_1 -> link3_1; origin xyz=-0.0025 -0.004186 0.0 rpy=0 0 0 -> xyz=0.0165 0.0 0.0 rpy=0 0 0; parent Adapter_B_1 -> cap2_1
- joint Rigid 45: child GearBox1_1 -> link3_leg2_1; origin xyz=-0.0093 0.004186 0.0 rpy=0 0 0 -> xyz=0.0 -0.10674 0.012 rpy=0 0 0; parent Adapter_A_1 -> link3_1
- joint Rigid 46: child Plug_1 -> link4_1; origin xyz=-0.1045 -0.004186 0.0 rpy=0 0 0 -> xyz=0.0 -0.194627 0.06 rpy=0 0 0; parent GearBox1_1 -> link3_1
- joint Rigid 47: child Link2_1_1 -> link5_1; origin xyz=0.0165 0.0 0.0 rpy=0 0 0 -> xyz=0.06865 0.0 0.0 rpy=0 0 0; parent Plug_1 -> link4_1
- joint Rigid 49: child Link2_1 -> motor2_1; origin xyz=0.1626 0.0 0.0 rpy=0 0 0 -> xyz=0.0039 0.005544 -0.0045 rpy=0 0 0; parent Link2Bridge_1 -> adapter_1
- joint Rigid 50: child Link2Bridge2_1 -> link2__1__1; origin xyz=0.0 0.0175 -0.092 rpy=0 0 0 -> xyz=-0.0067 0.005544 0.006 rpy=0 0 0; parent Link2_1 -> adapter_1
- joint Rigid 51: child Adapter_b_1_1 -> top_1; origin xyz=-0.004 0.144849 0.014 rpy=0 0 0 -> xyz=-0.005 -0.094 0.0035 rpy=0 0 0; parent Link2_1 -> link2__1__1
- joint Rigid 52: child Motor1_1 -> bottom_1; origin xyz=-0.0288 0.0 0.0 rpy=0 0 0 -> xyz=-0.005 -0.094 -0.013 rpy=0 0 0; parent Adapter_b_1_1 -> link2__1__1
- joint Rigid 62: child Motor2_1 -> link3-1_1; origin xyz=0.004 -0.063373 0.0 rpy=0 0 0 -> xyz=0.1943 0.0 0.0 rpy=0 0 0; parent Link_5_1 -> link3_leg_1
- joint Rigid 63: child Adapter_B_1_1_1 -> link4-1_1; origin xyz=0.0455 0.0 0.0 rpy=0 0 0 -> xyz=0.0 -0.087887 -0.048 rpy=0 0 0; parent Motor2_1 -> link3-1_1
- joint Rigid 64: child Link5_1_1 -> link5-1_1; origin xyz=0.0074 0.004186 0.0 rpy=0 0 0 -> xyz=-0.06865 0.0 0.0 rpy=0 0 0; parent Adapter_B_1_1_1 -> link4-1_1
- joint Rigid 65: child Link4_1_1 -> adapter_b__1___1__1; origin xyz=0.0 0.059187 0.0 rpy=0 0 0 -> xyz=0.0001 -0.068917 0.0045 rpy=0 0 0; parent Link5_1_1 -> link5-1_1
- joint joint_1: child Bottom_top_1 -> base_plate_1; limit (none) -> lower=-3.141593 upper=3.141593 effort=100 velocity=100; origin xyz=0.0 0.0 0.0505 rpy=0 0 0 -> xyz=0.0 0.0 0.0465 rpy=0 0 0; parent Motor0_1 -> lower_cylinder_1; type continuous -> revolute
- joint joint_2: axis -1.0 -0.0 0.0 -> -1.0 0.0 0.0; child Adapter_A_1 -> adapter_b_1; origin xyz=-0.048 0.0 0.0 rpy=0 0 0 -> xyz=0.0465 0.0 0.0 rpy=0 0 0; parent Motor_1 -> motor_1
- joint joint_3: child Adapter_A_1_1 -> cap2_1; limit lower=0.0 upper=3.665191 effort=100 velocity=100 -> lower=0.0 upper=3.141593 effort=100 velocity=100; origin xyz=-0.048 0.0 0.0 rpy=0 0 0 -> xyz=-0.0755 0.0 0.0 rpy=0 0 0; parent Motor1_1 -> gearbox1__1__1

Commit message: fix: Aug 19 검증 로봇 모델 복원

File: ros2_ws/src/robot_arm_description/urdf/robot_arm.urdf (robot description, URDF)
Before this commit: robot robot_arm, 44 links, 47 joints
Links:
- removed link ee_base_link
- added link link_042, mass 0.07583994930008672; collision mesh filename=package://robot_arm_description/meshes/link_042.stl scale=0.001 0.001 0.001; visual mesh filename=package://robot_arm_description/meshes/link_042.stl scale=0.001 0.001 0.001
- added link link_043, mass 0.5057750603466008; collision mesh filename=package://robot_arm_description/meshes/link_043.stl scale=0.001 0.001 0.001; visual mesh filename=package://robot_arm_description/meshes/link_043.stl scale=0.001 0.001 0.001
- added link link_044, mass 0.08821021033890362; collision mesh filename=package://robot_arm_description/meshes/link_044.stl scale=0.001 0.001 0.001; visual mesh filename=package://robot_arm_description/meshes/link_044.stl scale=0.001 0.001 0.001
- added link link_045, mass 0.08821021033890375; collision mesh filename=package://robot_arm_description/meshes/link_045.stl scale=0.001 0.001 0.001; visual mesh filename=package://robot_arm_description/meshes/link_045.stl scale=0.001 0.001 0.001
- added link link_046, mass 0.14107452059972816; collision mesh filename=package://robot_arm_description/meshes/link_046.stl scale=0.001 0.001 0.001; visual mesh filename=package://robot_arm_description/meshes/link_046.stl scale=0.001 0.001 0.001
- added link link_047, mass 0.14107452059972586; collision mesh filename=package://robot_arm_description/meshes/link_047.stl scale=0.001 0.001 0.001; visual mesh filename=package://robot_arm_description/meshes/link_047.stl scale=0.001 0.001 0.001
- added link link_048, mass 0.0034506939547765065; collision mesh filename=package://robot_arm_description/meshes/link_048.stl scale=0.001 0.001 0.001; visual mesh filename=package://robot_arm_description/meshes/link_048.stl scale=0.001 0.001 0.001
- added link link_049, mass 0.0034506939547765073; collision mesh filename=package://robot_arm_description/meshes/link_049.stl scale=0.001 0.001 0.001; visual mesh filename=package://robot_arm_description/meshes/link_049.stl scale=0.001 0.001 0.001
- added link link_050, mass 0.009342051864502975; collision mesh filename=package://robot_arm_description/meshes/link_050.stl scale=0.001 0.001 0.001; visual mesh filename=package://robot_arm_description/meshes/link_050.stl scale=0.001 0.001 0.001
Joints:
- removed joint wrist_to_ee
- added joint fixed_joint_038: type fixed, parent link_042, child link_043, origin xyz=0.014 -0.005 0.018 rpy=0 0 0
- added joint fixed_joint_039: type fixed, parent link_043, child link_044, origin xyz=-0.002 -0.034 -0.007 rpy=0 0 0
- added joint fixed_joint_040: type fixed, parent link_043, child link_045, origin xyz=-0.026 -0.034 -0.007 rpy=0 0 0
- added joint fixed_joint_041: type fixed, parent link_044, child link_048, origin xyz=0.008001 -0.002 -0.010249 rpy=0 0 0
- added joint fixed_joint_042: type fixed, parent link_045, child link_049, origin xyz=-0.007999 -0.0039 -0.01175 rpy=0 0 0
- joint arm_joint_2: limit lower=-0.2 upper=3.141593 effort=100 velocity=100 -> lower=0.0 upper=3.141593 effort=100 velocity=100
